Commit message: updates

File: src/wheelchair_navigation/urdf/wheelchair.urdf (robot description, URDF)
Before this commit: robot my_robot, 9 links, 8 joints
Links:
- link base_link: mass None -> 10.0; geometry collision box size=0.60 0.645 0.25; visual box size=0.04 0.40 0.55
- link left_front_caster: mass None -> 0.1; geometry collision sphere radius=0.05; visual sphere radius=0.05
- link left_rear_caster: mass None -> 0.1; geometry collision sphere radius=0.05; visual sphere radius=0.05
- link left_wheel: geometry collision cylinder length=0.05 radius=0.178; visual cylinder length=0.05 radius=0.178
- link right_front_caster: mass None -> 0.1; geometry collision sphere radius=0.05; visual sphere radius=0.05
- link right_rear_caster: mass None -> 0.1; geometry collision sphere radius=0.05; visual sphere radius=0.05
- link right_wheel: geometry collision cylinder length=0.05 radius=0.178; visual cylinder length=0.05 radius=0.178
Joints:
- joint base_joint: origin xyz=0 0 1.35 rpy=0 0 0 -> xyz=0 0 0.20 rpy=0 0 0

Commit message: rviz + single stereo camera using static odom shortcut to be fixed later

File: src/wheelchair_navigation/urdf/wheelchair.urdf (robot description, URDF)
Before this commit: robot wheelchair, 9 links, 8 joints
Links:
- removed link lidar_link
- added link camera_link, mass 0.1; collision box size=0.05 0.10 0.04; visual box size=0.05 0.10 0.04
Joints:
- removed joint lidar_joint
- added joint camera_joint: type fixed, parent base_link, child camera_link, origin xyz=0.30 0 0.20 rpy=0 0 0

Commit message: undid the bad thing

File: src/wheelchair_navigation/urdf/wheelchair.urdf (robot description, URDF)
Before this commit: robot wheelchair, 9 links, 8 joints
Links:
- removed link camera_link
- added link camera_back_left_link, mass 0.1; collision box size=0.05 0.10 0.04; visual box size=0.05 0.10 0.04
- added link camera_back_link, mass 0.1; collision box size=0.05 0.10 0.04; visual box size=0.05 0.10 0.04
- added link camera_back_right_link, mass 0.1; collision box size=0.05 0.10 0.04; visual box size=0.05 0.10 0.04
- added link camera_front_left_link, mass 0.1; collision box size=0.05 0.10 0.04; visual box size=0.05 0.10 0.04
- added link camera_front_link, mass 0.1; collision box size=0.05 0.10 0.04; visual box size=0.05 0.10 0.04
- added link camera_front_right_link, mass 0.1; collision box size=0.05 0.10 0.04; visual box size=0.05 0.10 0.04
Joints:
- removed joint camera_joint
- added joint camera_back_joint: type fixed, parent base_link, child camera_back_link, origin xyz=-0.30 0 0.20 rpy=0 0 3.14159
- added joint camera_back_left_joint: type fixed, parent base_link, child camera_back_left_link, origin xyz=-0.15 0.32 0.20 rpy=0 0 2.09
- added joint camera_back_right_joint: type fixed, parent base_link, child camera_back_right_link, origin xyz=-0.15 -0.32 0.20 rpy=0 0 -2.09
- added joint camera_front_joint: type fixed, parent base_link, child camera_front_link, origin xyz=0.30 0 0.20 rpy=0 0 0
- added joint camera_front_left_joint: type fixed, parent base_link, child camera_front_left_link, origin xyz=0.15 0.32 0.20 rpy=0 0 1.05
- added joint camera_front_right_joint: type fixed, parent base_link, child camera_front_right_link, origin xyz=0.15 -0.32 0.20 rpy=0 0 -1.05
